File: kicad/project.kicad_pcb (KiCad board)
At the start: 2 copper layers, 0 parts

Commit message: Inital footprints import
Parts:
- added C1: 10uF, Capacitors_SMD:C_0805_HandSoldering, F.Cu at (148.9, 107.1)
- added J1: CONN_01X04, Pin_Headers:Pin_Header_Straight_1x04_Pitch2.54mm, F.Cu at (138.6, 103.5)
- added J2: CONN_01X04, Pin_Headers:Pin_Header_Straight_1x04_Pitch2.54mm, F.Cu at (160.4, 103.2)
- added U1: APA102C, LEDs:LED_WS2812-PLCC6, F.Cu at (144.4, 101.3)
- added U2: APA102C, LEDs:LED_WS2812-PLCC6, F.Cu at (154.8, 103.0)
- added U3: APA102C, LEDs:LED_WS2812-PLCC6, F.Cu at (144.7, 112.0)
- added U4: APA102C, LEDs:LED_WS2812-PLCC6, F.Cu at (154.7, 112.3)
